File: Explore Labs 3D Gyroscope L3GD20H Breakout Board.brd (EAGLE design)
At the start: 20.4 x 20 mm, 27 parts, among them J2 M03, J3 M07-BOSCH, U1 L3GD20H, U2 MIC5365, U3 EXPLORE-LABS-LOGO-2-0.25

Commit message: clean up
Parts:
- J1: value M07-BOSCH -> M07-SENSOR
- Q1, Q2, Q3: value (none) -> 2N7002
- moved Q1 6.60 mm to (8.10, 8.90)
- moved Q3 6.60 mm to (8.10, 2.30)
- moved R1 4.43 mm to (5.90, 8.40)
- moved R2 4.43 mm to (5.90, 5.10)
- moved R3 4.43 mm to (5.90, 1.80)
- moved R4 4.43 mm to (10.3, 8.90)
- moved R5 4.43 mm to (10.3, 5.60)
- moved R6 4.43 mm to (10.3, 2.30)
- renumbered J3 to J1, LOGO2 to ZZ2, Q4 to Q2, U$1 to ZZ3, U$8 to ZZ4, U3 to ZZ1
Connections:
- net CS_H: now also Q3.3, R3.1; no longer Q1.3, R6.1
- net CS_L: now also Q3.2, R6.1; no longer Q1.2, R3.1
- net SCK_H: now also R2.1; no longer R5.1
- net SCK_L: now also R5.1; no longer R2.1
- net SDI_H: now also Q1.3, R1.1; no longer Q3.3, R4.1
- net SDI_L: now also Q1.2, R4.1; no longer Q3.2, R1.1
- net VDD: now also R4.2, R5.2, R6.2; no longer R1.2, R2.2, R3.2
- net VIN: now also R1.2, R2.2, R3.2; no longer R4.2, R5.2, R6.2
