File: Explore Labs 3D Gyroscope L3GD20H Breakout Board.sch (EAGLE design)
At the start: 27 parts, among them J2 M03, J3 M07-BOSCH, U1 L3GD20H, U2 MIC5365, U3 EXPLORE-LABS-LOGO-2-0.25

Commit message: clean up
Parts:
- removed J3: M07-BOSCH, Explore Labs EAGLE Library:M07-BOSCH
- added J1: M07-SENSOR, Explore Labs EAGLE Library:M07-SENSOR
- Q1, Q2, Q3: value (none) -> 2N7002
- renumbered LOGO2 to ZZ2, Q4 to Q2, U$1 to ZZ3, U$8 to ZZ4, U3 to ZZ1
Connections:
- net CS_H: now also J1.7, Q3.D, R3.1; no longer J3.7, Q1.D, R6.1
- net CS_L: now also Q3.S, R6.1; no longer Q1.S, R3.1
- net GND: now also J1.3; no longer J3.3
- net SCK_H: now also J1.5, R2.1; no longer J3.5, R5.1
- net SCK_L: now also R5.1; no longer R2.1
- net SDI_H: now also J1.4, Q1.D, R1.1; no longer J3.4, Q3.D, R4.1
- net SDI_L: now also Q1.S, R4.1; no longer Q3.S, R1.1
- net SDO_L: now also J1.6; no longer J3.6
- net VDD: now also J1.2, R4.2, R5.2, R6.2; no longer J3.2, R1.2, R2.2, R3.2
- net VIN: now also J1.1, R1.2, R2.2, R3.2; no longer J3.1, R4.2, R5.2, R6.2
Other:
- note added: "DEN_L INT1_L INT2_L (Not level shifted)"
- note added: "Explore Labs 3D Gyroscope L3GD20H Breakout Board"
- note removed: "INT1 INT2 DEN_L not level shifted"
- moved on the sheet: Q1, Q3, R1, R2, R3, R4, R5, R6
